Commit message: launch sim in gazebo

File: description/gazebo_control.xacro (robot description, xacro)
@@ -3,4 +3,7 @@
     <gazebo>
         <plugin name="diff_drive" filename="libgazebo_ros_diff_drive.so">
+    <alwaysOn>true</alwaysOn>
+    <legacyMode>false</legacyMode>
+    <updateRate>40</updateRate>
             <!-- Wheel Information -->
             <left_joint>left_wheel_joint</left_joint>
@@ -12,4 +15,5 @@
             <max_wheel_acceleration>10.0</max_wheel_acceleration>
             <!-- Output -->
+            <commandTopic>cmd_vel</commandTopic>
             <odometry_frame>odom</odometry_frame>
             <robot_base_frame>base_link</robot_base_frame>

File: description/rover.urdf.xacro (robot description, xacro)
@@ -1,12 +1,12 @@
 <?xml version="1.0"?>
-<robot xmlns:xacro="http://www.ros.org/wiki/xacro"  name="robot">
+<robot xmlns:xacro="http://www.ros.org/wiki/xacro" name="rover">
     <xacro:arg name="use_ros2_control" default="true"/>
     <xacro:arg name="sim_mode" default="false"/>
     <xacro:include filename="rover_core.xacro" />
-    <xacro:if value="$(arg use_ros2_control)">
+    <!--xacro:if value="$(arg use_ros2_control)">
         <xacro:include filename="ros2_control.xacro" />
-    </xacro:if>
-    <xacro:unless value="$(arg use_ros2_control)">
+    </xacro:if-->
+    <!--xacro:unless value="$(arg use_ros2_control)"-->
         <xacro:include filename="gazebo_control.xacro" />
-    </xacro:unless>
+    <!--/xacro:unless-->
 </robot>

File: description/rover.xacro (robot description, xacro)
@@ -30,5 +30,5 @@
       <origin rpy="0 0 0" xyz="0.03 0 -0.026"/>
       <geometry>
-        <mesh filename="package://rover_ctrl/meshes/Chasis.stl" scale="0.001 0.001 0.001"/>
+        <mesh filename="file://$(find rover_ctrl)/meshes/Chasis.stl" scale="0.001 0.001 0.001"/>
       </geometry>
       <material name="olivegreen"/>
@@ -37,5 +37,5 @@
       <origin rpy="0 0 0" xyz="0.03 0 -0.026" />
       <geometry>
-        <mesh filename="package://rover_ctrl/meshes/Chasis.stl" scale="0.001 0.001 0.001" />
+        <mesh filename="file://$(find rover_ctrl)/meshes/Chasis.stl" scale="0.001 0.001 0.001" />
       </geometry>
     </collision>
@@ -50,5 +50,5 @@
       <origin rpy="0 0 -1.5708" xyz="0.084 -0.242 -0.098"/>
       <geometry>
-        <mesh filename="package://rover_ctrl/meshes/RpLidar.stl" scale="0.001 0.001 0.001"/>
+        <mesh filename="file://$(find rover_ctrl)/meshes/RpLidar.stl" scale="0.001 0.001 0.001"/>
       </geometry>
       <material name="blue"/>
@@ -57,5 +57,5 @@
       <origin rpy="0 0 0" xyz="0.242 0.084 -0.098" />
       <geometry>
-        <mesh filename="package://rover_ctrl/meshes/RpLidar.stl" scale="0.001 0.001 0.001" />
+        <mesh filename="file://$(find rover_ctrl)/meshes/RpLidar.stl" scale="0.001 0.001 0.001" />
       </geometry>
     </collision>
@@ -72,5 +72,5 @@
         <origin rpy="0 0 0" xyz="${x} 0.059 -0.04"/>
         <geometry>
-          <mesh filename="package://rover_ctrl/meshes/Wheel.stl" scale="0.001 0.001 0.001"/>
+          <mesh filename="file://$(find rover_ctrl)/meshes/Wheel.stl" scale="0.001 0.001 0.001"/>
         </geometry>
         <material name="black"/>
@@ -79,5 +79,5 @@
         <origin rpy="0 0 0" xyz="${x} 0.059 -0.04"/>
         <geometry>
-          <mesh filename="package://rover_ctrl/meshes/Wheel.stl" scale="0.001 0.001 0.001" />
+          <mesh filename="file://$(find rover_ctrl)/meshes/Wheel.stl" scale="0.001 0.001 0.001" />
         </geometry>
       </collision>

File: description/rover_core.xacro (robot description, xacro)
@@ -12,4 +12,8 @@
     <xacro:property name="wheel_offset_y" value="0.1485"/>
     <xacro:property name="wheel_offset_z" value="0.01"/>
+    <xacro:property name="caster_wheel_radius" value="0.01"/>
+    <xacro:property name="caster_wheel_mass" value="0.01"/>
+    <xacro:property name="caster_wheel_offset_x" value="0.006557"/>
+    <xacro:property name="caster_wheel_offset_z" value="0.097098"/>
     <material name="white">
         <color rgba="1 1 1 1" />
@@ -120,4 +124,31 @@
         <turnGravityOff>true</turnGravityOff>
     </gazebo>
+<!-- CASTER WHEEL LINK -->
+    <joint name="caster_wheel_joint" type="fixed">
+        <parent link="chassis"/>
+        <child link="caster_wheel"/>
+        <origin xyz="${caster_wheel_offset_x} 0 ${caster_wheel_offset_z}"/>
+    </joint>
+    <link name="caster_wheel">
+        <visual>
+            <geometry>
+                <sphere radius="${caster_wheel_radius}"/>
+            </geometry>
+            <material name="white"/>
+        </visual>
+        <collision>
+            <geometry>
+                <sphere radius="${caster_wheel_radius}"/>
+            </geometry>
+        </collision>
+        <xacro:inertial_sphere mass="${caster_wheel_mass}" radius="${caster_wheel_radius}">
+            <origin xyz="0 0 0" rpy="0 0 0"/>
+        </xacro:inertial_sphere>
+    </link>
+    <gazebo reference="caster_wheel">
+        <material>Gazebo/White</material>
+        <mu1 value="0.001"/>
+        <mu2 value="0.001"/>
+    </gazebo>
     <!-- LIDAR LINK -->
     <joint name="laser_joint" type="fixed">
