Commit message: update project deps

File: description/bot_arch.xacro (robot description, xacro)
@@ -6,5 +6,5 @@
     <xacro:property name="chassis_height" value="0.138"/>
     <xacro:property name="chassis_mass" value="1.0"/>
-    <xacro:property name="wheel_radius" value="0.04"/>
+    <xacro:property name="wheel_radius" value="0.033"/>
     <xacro:property name="wheel_thickness" value="0.026"/>
     <xacro:property name="wheel_mass" value="0.05"/>
@@ -14,11 +14,11 @@
     <xacro:property name="caster_wheel_radius" value="0.01"/>
     <xacro:property name="caster_wheel_mass" value="0.01"/>
-    <xacro:property name="caster_wheel_offset_x" value="0.006557"/>
-    <xacro:property name="caster_wheel_offset_z" value="0.097098"/>
+    <xacro:property name="caster_wheel_offset_x" value="0.075"/>
+    <xacro:property name="caster_wheel_offset_z" value="${wheel_offset_z - wheel_radius + caster_wheel_radius}"/>
     <material name="white">
         <color rgba="1 1 1 1" />
     </material>
-    <material name="olivegreen">
-        <color rgba="0.729 0.722 0.424 1.0"/>
+    <material name="orange">
+        <color rgba="1 0.3 0.1 1"/>
     </material>
     <material name="blue">
@@ -28,59 +28,62 @@
         <color rgba="0 0 0 1"/>
     </material>
+    <material name="red">
+        <color rgba="1 0 0 1"/>
+    </material>
     <!-- BASE LINK -->
     <link name="base_link">
-        <collision>
-            <origin rpy="0 0 0" xyz="0 0 0.0005"/>
-            <geometry>
-                <box size="0.22 0.22 0.001"/>
-            </geometry>
-        </collision>
-    </link>
-    <joint name="base_link_joint" type="fixed">
-        <origin rpy="0 0 -1.5708" xyz="0 0 0.026"/>
+    </link>
+    <!-- BASE_FOOTPRINT LINK -->
+    <joint name="base_footprint_joint" type="fixed">
+        <parent link="base_link"/>
+        <child link="base_footprint"/>
+        <origin xyz="0 0 0" rpy="0 0 0"/>
+    </joint>
+    <link name="base_footprint">
+    </link>
+    <!-- CHASSIS LINK -->
+    <joint name="chassis_joint" type="fixed">
         <parent link="base_link"/>
         <child link="chassis"/>
-    </joint>
-    <!-- CHASSIS LINK -->
+        <origin xyz="${-wheel_offset_x} 0 ${-wheel_offset_z}"/>
+    </joint>
     <link name="chassis">
         <visual>
-            <origin rpy="0 0 0" xyz="0.03 0 -0.02"/>
-            <geometry>
-                <mesh filename="file://$(find rover_ctrl)/meshes/Chasis.stl" scale="0.001 0.001 0.001"/>
-            </geometry>
-            <material name="olivegreen"/>
-        </visual>
-        <collision>
-            <origin rpy="0 0 0" xyz="0.03 0 -0.02"/>
-            <geometry>
-                <mesh filename="file://$(find rover_ctrl)/meshes/Chasis.stl" scale="0.001 0.001 0.001"/>
-            </geometry>
-        </collision>
-        <xacro:inertial_box mass="${chassis_mass}" x="${chassis_length}" y="${chassis_width}" z="${chassis_height}" >
-            <origin xyz="0 0 0" rpy="0 0 0"/>
+            <origin xyz="${chassis_length/2} 0 ${chassis_height/2}"/>
+            <geometry>
+                <box size="${chassis_length} ${chassis_width} ${chassis_height}"/>
+            </geometry>
+            <material name="orange"/>
+        </visual>
+        <collision>
+            <origin xyz="${chassis_length/2} 0 ${chassis_height/2}"/>
+            <geometry>
+                <box size="${chassis_length} ${chassis_width} ${chassis_height}"/>
+            </geometry>
+        </collision>
+        <xacro:inertial_box mass="0.5" x="${chassis_length}" y="${chassis_width}" z="${chassis_height}">
+            <origin xyz="${chassis_length/2} 0 ${chassis_height/2}" rpy="0 0 0"/>
         </xacro:inertial_box>
     </link>
     <gazebo reference="chassis">
-        <material>Gazebo/Green</material>
+        <material>Gazebo/Orange</material>
     </gazebo>
     <!-- LEFT WHEEL LINK -->
     <joint name="left_wheel_joint" type="continuous">
-        <parent link="chassis"/>
+        <parent link="base_link"/>
         <child link="left_wheel"/>
-        <origin rpy="0 0 0" xyz="0.08 -0.06 0"/>
-        <axis xyz="-1 0 0"/>
+        <origin xyz="0 ${wheel_offset_y} 0" rpy="-${pi/2} 0 0" />
+        <axis xyz="0 0 1"/>
     </joint>
     <link name="left_wheel">
         <visual>
-            <origin rpy="0 0 0" xyz="0.133 0.059 -0.0435"/>
-            <geometry>
-                <mesh filename="file://$(find rover_ctrl)/meshes/Wheel.stl" scale="0.001 0.001 0.001"/>
+            <geometry>
+                <cylinder radius="${wheel_radius}" length="${wheel_thickness}"/>
             </geometry>
             <material name="black"/>
         </visual>
         <collision>
-            <origin rpy="0 0 0" xyz="0.133 0.059 -0.0435"/>
-            <geometry>
-                <mesh filename="file://$(find rover_ctrl)/meshes/Wheel.stl" scale="0.001 0.001 0.001"/>
+            <geometry>
+                <sphere radius="${wheel_radius}"/>
             </geometry>
         </collision>
@@ -94,22 +97,19 @@
     <!-- RIGHT WHEEL LINK -->
     <joint name="right_wheel_joint" type="continuous">
-        <parent link="chassis"/>
+        <parent link="base_link"/>
         <child link="right_wheel"/>
-        <!-- origin xyz="0 ${-wheel_offset_y} 0" rpy="${pi/2} 0 0" / -->
-        <origin rpy="0 0 0" xyz="-0.08 -0.06 0"/>
-        <axis xyz="-1 0 0"/>
+        <origin xyz="0 ${-wheel_offset_y} 0" rpy="${pi/2} 0 0" />
+        <axis xyz="0 0 -1"/>
     </joint>
     <link name="right_wheel">
         <visual>
-            <origin rpy="0 0 0" xyz="0.11 0.059 -0.045"/>
-            <geometry>
-                <mesh filename="file://$(find rover_ctrl)/meshes/Wheel.stl" scale="0.001 0.001 0.001"/>
+            <geometry>
+                <cylinder radius="${wheel_radius}" length="${wheel_thickness}"/>
             </geometry>
             <material name="black"/>
         </visual>
         <collision>
-            <origin rpy="0 0 0" xyz="0.11 0.059 -0.045"/>
-            <geometry>
-                <mesh filename="file://$(find rover_ctrl)/meshes/Wheel.stl" scale="0.001 0.001 0.001"/>
+            <geometry>
+                <sphere radius="${wheel_radius}"/>
             </geometry>
         </collision>
@@ -121,23 +121,54 @@
         <material>Gazebo/Black</material>
     </gazebo>
-	<!-- CASTER WHEEL LINK -->
+    <!-- CASTER WHEEL LINK -->
+    <joint name="caster_wheel_joint" type="fixed">
+        <parent link="chassis"/>
+        <child link="caster_wheel"/>
+        <origin xyz="${caster_wheel_offset_x} 0 ${caster_wheel_offset_z}"/>
+    </joint>
+    <link name="caster_wheel">
+        <visual>
+            <geometry>
+                <sphere radius="${caster_wheel_radius}"/>
+            </geometry>
+            <material name="white"/>
+        </visual>
+        <collision>
+            <geometry>
+                <sphere radius="${caster_wheel_radius}"/>
+            </geometry>
+        </collision>
+        <xacro:inertial_sphere mass="${caster_wheel_mass}" radius="${caster_wheel_radius}">
+            <origin xyz="0 0 0" rpy="0 0 0"/>
+        </xacro:inertial_sphere>
+    </link>
+    <gazebo reference="caster_wheel">
+        <material>Gazebo/White</material>
+        <mu1 value="0.001"/>
+        <mu2 value="0.001"/>
+    </gazebo>
     <!-- LIDAR LINK -->
     <joint name="laser_joint" type="fixed">
         <parent link="chassis"/>
         <child link="laser_frame"/>
-        <origin rpy="0 0 1.5708" xyz="0 0.040 0.090"/>
+        <origin xyz="0.122 0 0.212" rpy="0 0 0"/>
     </joint>
     <link name="laser_frame">
         <visual>
-            <origin rpy="0 0 -1.5708" xyz="0.084 -0.242 -0.09"/>
-            <geometry>
-                <mesh filename="file://$(find rover_ctrl)/meshes/RpLidar.stl" scale="0.001 0.001 0.001"/>
+            <geometry>
+                <cylinder radius="0.05" length="0.04"/>
             </geometry>
             <material name="blue"/>
         </visual>
-        <collision>
-            <origin rpy="0 0 0" xyz="0.242 0.084 -0.09"/>
-            <geometry>
-                <mesh filename="file://$(find rover_ctrl)/meshes/RpLidar.stl" scale="0.001 0.001 0.001"/>
+        <visual>
+            <origin xyz="0 0 -0.05"/>
+            <geometry>
+                <cylinder radius="0.01" length="0.1"/>
+            </geometry>
+            <material name="blue"/>
+        </visual>
+        <collision>
+            <geometry>
+                <cylinder radius="0.05" length="0.04"/>
             </geometry>
         </collision>
@@ -148,4 +179,29 @@
     <gazebo reference="laser_frame">
         <material>Gazebo/Blue</material>
+        <sensor name="laser" type="ray">
+            <pose> 0 0 0 0 0 0 </pose>
+            <visualize>true</visualize>
+            <update_rate>10</update_rate>
+            <ray>
+                <scan>
+                    <horizontal>
+                        <samples>360</samples>
+                        <min_angle>-3.14</min_angle>
+                        <max_angle>3.14</max_angle>
+                    </horizontal>
+                </scan>
+                <range>
+                    <min>0.3</min>
+                    <max>12</max>
+                </range>
+            </ray>
+            <plugin name="laser_controller" filename="libgazebo_ros_ray_sensor.so">
+                <ros>
+                    <remapping>~/out:=scan</remapping>
+                </ros>
+                <output_type>sensor_msgs/LaserScan</output_type>
+                <frame_name>laser_frame</frame_name>
+            </plugin>
+        </sensor>
     </gazebo>
 </robot>

File: description/rover.urdf.xacro (robot description, xacro)
@@ -2,11 +2,23 @@
 <robot xmlns:xacro="http://www.ros.org/wiki/xacro" name="rover">
     <xacro:arg name="use_ros2_control" default="true"/>
-    <xacro:arg name="sim_mode" default="false"/>
+    <xacro:arg name="sim_mode" default="true"/>
     <xacro:include filename="bot_arch.xacro" />
-    <!--xacro:if value="$(arg use_ros2_control)">
-        <xacro:include filename="ros2_control.xacro" />
-    </xacro:if-->
-    <!--xacro:unless value="$(arg use_ros2_control)"-->
-        <xacro:include filename="gz_ctrl.xacro" />
-    <!--/xacro:unless-->
+    <gazebo>
+        <plugin name="diff_drive" filename="libgazebo_ros_diff_drive.so">
+            <!-- Wheel Information -->
+            <left_joint>left_wheel_joint</left_joint>
+            <right_joint>right_wheel_joint</right_joint>
+            <wheel_separation>0.297</wheel_separation>
+            <wheel_diameter>0.066</wheel_diameter>
+            <!-- Limits -->
+            <max_wheel_torque>200</max_wheel_torque>
+            <max_wheel_acceleration>10.0</max_wheel_acceleration>
+            <!-- Output -->
+            <odometry_frame>odom</odometry_frame>
+            <robot_base_frame>base_link</robot_base_frame>
+            <publish_odom>true</publish_odom>
+            <publish_odom_tf>true</publish_odom_tf>
+            <publish_wheel_tf>true</publish_wheel_tf>
+        </plugin>
+    </gazebo>
 </robot>
